Commit message: feat: integrate visual grasp and hardware safety workflow

File: src/rebotarm_bringup/description/urdf/reBot-DevArm_fixend.urdf (robot description, URDF)
Before this commit: robot reBot-DevArm_fixend, 10 links, 9 joints
Joints:
- joint joint2: limit lower=-3.14 upper=0 effort=27 velocity=50 -> lower=-3.14 upper=0.02 effort=27 velocity=50

File: src/rebotarm_moveit_config/config/rebotarm.urdf (robot description, URDF)
Before this commit: robot reBot-DevArm_fixend, 10 links, 9 joints
Joints:
- joint joint2: limit lower=-3.14 upper=0 effort=27 velocity=50 -> lower=-3.14 upper=0.02 effort=27 velocity=50
