Commit message: fix: align joint3 upper margin across hardware and models

File: src/rebotarm_moveit_config/config/rebotarm.urdf (robot description, URDF)
Before this commit: robot reBot-DevArm_fixend, 10 links, 9 joints
Joints:
- joint joint3: limit lower=-3.14 upper=0 effort=27 velocity=50 -> lower=-3.14 upper=0.02 effort=27 velocity=50
